Commit message: removed schmalz_ecbpmi and replaced mesh with a dummy box

File: src/irc_ros_description/urdf/grippers/ext_dio_gripper.description.xacro (robot description, xacro)
@@ -34,5 +34,8 @@
       <visual>
         <geometry>
-          <mesh filename="file://$(find irc_ros_description)/meshes/gripper_schmalz_ecbpmi/Joint0.dae"/>
+          <!-- Original mesh, now commented -->
+          <!-- <mesh filename="file://$(find irc_ros_description)/meshes/..."/> -->
+          <!-- Replaced with a box -->
+          <box size="0.1 0.1 0.1"/>
         </geometry>
         <origin rpy="0.0 0.0 ${pi/2}" xyz="0.07 0.0 0.0"/>
@@ -40,5 +43,7 @@
       <collision>
         <geometry>
-          <mesh filename="file://$(find irc_ros_description)/meshes/gripper_schmalz_ecbpmi/Joint0Coll.dae"/>
+          <!-- <mesh filename="file://$(find irc_ros_description)/meshes/..."/> -->
+          <!-- Replaced with a box -->
+          <box size="0.1 0.1 0.1"/>
         </geometry>
         <origin rpy="0.0 0.0 ${pi/2}" xyz="0.07 0.0 0.0"/>

File: src/irc_ros_description/urdf/grippers/grippers.macro.xacro (robot description, xacro)
@@ -5,5 +5,4 @@
   <xacro:include filename="$(find irc_ros_description)/urdf/grippers/ext_dio_gripper.description.xacro" />
   <xacro:include filename="$(find irc_ros_description)/urdf/grippers/ext_dio_gripper.ros2_control.xacro" />
-  <xacro:include filename="$(find irc_ros_description)/urdf/grippers/schmalz_ecbpmi.description.xacro" />
   <xacro:macro name="gripper" params="prefix gripper_type parent_link hardware_protocol">
     <!-- Call macros once -->
@@ -11,7 +10,4 @@
       <xacro:ext_dio_gripper_description prefix="${prefix}" parent_link="${parent_link}" />
       <xacro:ext_dio_gripper_ros2_control prefix="${prefix}" parent_link="${parent_link}" hardware_protocol="${hardware_protocol}" />
-    </xacro:if>
-    <xacro:if value="${gripper_type == 'schmalz_ecbpmi'}">
-      <xacro:schmalz_ecbpmi_description prefix="${prefix}" parent_link="${parent_link}" />
     </xacro:if>
     <xacro:if value="${gripper_type == 'none'}">
